Commit message: Changes got robot model on rviz

File: sim_tutorial/description/urdf/cybertruck.urdf.xacro (robot description, xacro)
@@ -3,5 +3,12 @@
   <link name="base_link"/>
   <!-- Your URDF code here -->
-  <link name="body_link"/>
+  <link name="body_link">
+    <visual>
+          <origin xyz="0 0 0" rpy="0 0 0"/>
+            <geometry>
+               <mesh filename="package://description/urdf/meshes/cybertruck_body.dae"/>
+            </geometry>
+    </visual>
+  </link>
   <joint name="body_joint" type="fixed">
     <parent link="base_link"/>

Commit message: added wheels. Works in Rviz

File: sim_tutorial/description/urdf/cybertruck.urdf.xacro (robot description, xacro)
@@ -10,4 +10,10 @@
             </geometry>
     </visual>
+    <collision>
+            <origin xyz="0 0 0" rpy="0 0 0"/>
+            <geometry>
+               <mesh filename="package://description/urdf/meshes/cybertruck_body.dae"/>
+            </geometry>
+    </collision>
   </link>
   <joint name="body_joint" type="fixed">
@@ -16,3 +22,5 @@
     <origin xyz="0 0 0 " rpy="0 0 ${pi / 2}"/>
   </joint>
+  <!--Wheels-->
+    <xacro:include filename="$(find description)/urdf/wheels.urdf.xacro"/>
 </robot>

Commit message: Works in Rviz and Gazebo

File: sim_tutorial/description/urdf/cybertruck.urdf.xacro (robot description, xacro)
@@ -1,4 +1,7 @@
 <?xml version="1.0"?>
 <robot name="file_name" xmlns:xacro="http://ros.org/wiki/xacro">
+  <!--Includes-->
+  <xacro:include filename="$(find description)/urdf/constants.xacro"/>
+  <xacro:include filename="$(find description)/urdf/inertias.xacro"/>
   <link name="base_link"/>
   <!-- Your URDF code here -->
@@ -16,4 +19,7 @@
             </geometry>
     </collision>
+    <inertia>
+      <xacro:body_inertial m="${body_mass}" l="${body_length}" w="${body_width}" h="${body_height}"/>
+    </inertia>
   </link>
   <joint name="body_joint" type="fixed">

File: sim_tutorial/description/urdf/wheels.urdf.xacro (robot description, xacro)
@@ -22,5 +22,6 @@
             <parent link="body_link"/>
             <child link="${fb}_${lr}_wheel_link"/>
-            <origin xyz="${left_wheel if lr == 'left' else right_wheel} ${front_wheel if fb == 'front' else back_wheel} ${height_to_wheel} " rpy="0 0 0"/>
+            <origin xyz="${left_wheel if lr == 'left' else right_wheel} ${front_wheel if fb == 'front' else back_wheel} ${height_to_wheel}" rpy="0 0 0"/>
+            <axis xyz="1 0 0"/>
         </joint>
     </xacro:macro>

Commit message: Full Robot Spawned in Gazebo

File: sim_tutorial/description/urdf/cybertruck.urdf.xacro (robot description, xacro)
@@ -4,4 +4,5 @@
   <xacro:include filename="$(find description)/urdf/constants.xacro"/>
   <xacro:include filename="$(find description)/urdf/inertias.xacro"/>
+  <!--xacro:include filename="$(find description)/urdf/plugins.gazebo.xacro"/-->
   <link name="base_link"/>
   <!-- Your URDF code here -->
@@ -19,7 +20,7 @@
             </geometry>
     </collision>
-    <inertia>
+    <inertial>
       <xacro:body_inertial m="${body_mass}" l="${body_length}" w="${body_width}" h="${body_height}"/>
-    </inertia>
+    </inertial>
   </link>
   <joint name="body_joint" type="fixed">
@@ -30,3 +31,10 @@
   <!--Wheels-->
     <xacro:include filename="$(find description)/urdf/wheels.urdf.xacro"/>
+  <!--LIDAR>
+    <link name="scan_link"/>
+    <joint name="body_joint" type="fixed">
+      <parent link="body_link"/>
+      <child link="scan_link"/>
+      <origin xyz="0 ${front_wheel} ${-height_to_wheel} " rpy="0 0 ${-pi / 2}"/>
+   </joint-->
 </robot>

File: sim_tutorial/description/urdf/inertias.xacro (robot description, xacro)
@@ -14,3 +14,11 @@
     <!-- NOTE: wheels are radially symmetric around the x-axis -->
     <!-- TODO: define a macro for the inertial of a wheel (can approx as a cylinder) -->
+    <xacro:macro name="wheel_inertial" params="m r h">
+        <mass value="${m}"/>
+        <inertia
+            ixx="${m*r*r/2}" ixy="0" ixz="0"
+            iyy="${m*(3*r*r + h*h)/12}" iyz="0"
+            izz="${m*(3*r*r + h*h)/12}"
+        />
+    </xacro:macro>
 </robot>

File: sim_tutorial/description/urdf/wheels.urdf.xacro (robot description, xacro)
@@ -18,4 +18,7 @@
                 </geometry>
             </collision>
+            <inertial>
+                <xacro:wheel_inertial m="${wheel_mass}" r="${wheel_radius}" h="${wheel_width}"/>
+            </inertial>
         </link>
         <joint name="${fb}_${lr}_wheel_joint" type="continuous">
